File: catboard/catboard.kicad_sch (KiCad schematic)
At the start: 19 parts, among them J1 USB_C_Receptacle_USB2.0_14P, U1 RP2040, U2 MCP1700x-330xxTT

Commit message: badeep
Parts:
- added C15, C16: 15pF, symbol Device:C
- added C17: 0.1uF, symbol Device:C
- added J2, J3: Conn_01x20, symbol Connector_Generic:Conn_01x20
- added J4: Conn_01x03, symbol Connector_Generic:Conn_01x03
- added R3, R4: 27, symbol Device:R
- added R5: R, symbol Device:R
- added R6: 10k, symbol Device:R
- added R7: 1k, symbol Device:R
- added SW1: SW_Push, symbol Switch:SW_Push
- added U3: W25Q128JVS, Package_SO:SOIC-8_5.3x5.3mm_P1.27mm, symbol Memory_Flash:W25Q128JVS
- added Y1: 12 MHz, symbol Device:Crystal_GND24
Connections:
- net +3V3: now also C17.1, J3.5 (Pin_5), R6.1, U3.8 (VCC)
- net GND: now also U1.19 (TESTEN), C15.1, C16.1, C17.2, J2.13 (Pin_13), J2.18 (Pin_18), J2.3 (Pin_3), J2.8 (Pin_8), J3.13 (Pin_13), J3.18 (Pin_18), J3.3 (Pin_3), J3.8 (Pin_8), J4.2 (Pin_2), SW1.1, U3.4 (GND), Y1.2 (G), Y1.4 (G)
- net USB_D+: now also R4.2
- net USB_D-: now also R3.2
- net VBUS: now also J3.1 (Pin_1)
- net GPI8: now reaches U1.11 (GPIO8)
- net GPI8: now also J2.11 (Pin_11)
- net GPI9: now reaches U1.12 (GPIO9)
- net GPI9: now also J2.12 (Pin_12)
- net GPI10: now reaches U1.13 (GPIO10)
- net GPI10: now also J2.14 (Pin_14)
- net GPI11: now reaches U1.14 (GPIO11)
- net GPI11: now also J2.15 (Pin_15)
- net GPI12: now reaches U1.15 (GPIO12)
- net GPI12: now also J2.16 (Pin_16)
- net GPI13: now reaches U1.16 (GPIO13)
- net GPI13: now also J2.17 (Pin_17)
- net GPI14: now reaches U1.17 (GPIO14)
- net GPI14: now also J2.19 (Pin_19)
- net GPI15: now reaches U1.18 (GPIO15)
- net GPI15: now also J2.20 (Pin_20)
- net GPI0: now reaches U1.2 (GPIO0)
- net GPI0: now also J2.1 (Pin_1)
- net XIN: now reaches U1.20 (XIN)
- net XIN: now also C15.2, Y1.3
- net XOUT: now reaches U1.21 (XOUT)
- net XOUT: now also R5.1
- net SWCLK: now reaches U1.24 (SWCLK)
- net SWCLK: now also J4.1 (Pin_1)
- net SWD: now reaches U1.25 (SWDIO)
- net SWD: now also J4.3 (Pin_3)
- net RUN: now reaches U1.26 (RUN)
- net RUN: now also J3.11 (Pin_11)
- net GPI16: now reaches U1.27 (GPIO16)
- net GPI16: now also J3.20 (Pin_20)
- net GPI17: now reaches U1.28 (GPIO17)
- net GPI17: now also J3.19 (Pin_19)
- net GPI18: now reaches U1.29 (GPIO18)
- net GPI18: now also J3.17 (Pin_17)
- net GPI1: now reaches U1.3 (GPIO1)
- net GPI1: now also J2.2 (Pin_2)
- net GPI19: now reaches U1.30 (GPIO19)
- net GPI19: now also J3.16 (Pin_16)
- net GPI20: now reaches U1.31 (GPIO20)
- net GPI20: now also J3.15 (Pin_15)
- net GPI21: now reaches U1.32 (GPIO21)
- net GPI21: now also J3.14 (Pin_14)
- net GPI22: now reaches U1.34 (GPIO22)
- net GPI22: now also J3.12 (Pin_12)
- net GPI23: now reaches U1.35 (GPIO23)
- net GPI23: now also J3.10 (Pin_10)
- net GPI24: now reaches U1.36 (GPIO24)
- net GPI24: now also J3.9 (Pin_9)
- net GPI26_ADC0: now reaches U1.38 (GPIO26/ADC0)
- net GPI26_ADC0: now also J3.7 (Pin_7)
- net GPI27_ADC1: now reaches U1.39 (GPIO27/ADC1)
- net GPI27_ADC1: now also J3.6 (Pin_6)
- net GPI2: now reaches U1.4 (GPIO2)
- net GPI2: now also J2.4 (Pin_4)
- net GPI28_ADC2: now reaches U1.40 (GPIO28/ADC2)
- net GPI28_ADC2: now also J3.4 (Pin_4)
- net GPI29_ADC3: now reaches U1.41 (GPIO29/ADC3)
- net GPI29_ADC3: now also J3.2 (Pin_2)
- net at U1.46 (USB_DM): now also R3.1
- net at U1.47 (USB_DP): now also R4.1
- net GPI3: now reaches U1.5 (GPIO3)
- net GPI3: now also J2.5 (Pin_5)
- net QSPI_SD3: now reaches U1.51 (QSPI_SD3)
- net QSPI_SD3: now also U3.7 (~{HOLD}/~{RESET}/IO_{3})
- net QSPI_SCLK: now reaches U1.52 (QSPI_SCLK)
- net QSPI_SCLK: now also U3.6 (CLK)
- net QSPI_SD0: now reaches U1.53 (QSPI_SD0)
- net QSPI_SD0: now also U3.5 (DI/IO_{0})
- net QSPI_SD2: now reaches U1.54 (QSPI_SD2)
- net QSPI_SD2: now also U3.3 (~{WP}/IO_{2})
- net QSPI_SD1: now reaches U1.55 (QSPI_SD1)
- net QSPI_SD1: now also U3.2 (DO/IO_{1})
- net QSPI_SS: now reaches U1.56 (~{QSPI_SS})
- net QSPI_SS: now also R6.2, R7.2, U3.1 (~{CS})
- net GPI4: now reaches U1.6 (GPIO4)
- net GPI4: now also J2.6 (Pin_6)
- net GPI5: now reaches U1.7 (GPIO5)
- net GPI5: now also J2.7 (Pin_7)
- net GPI6: now reaches U1.8 (GPIO6)
- net GPI6: now also J2.9 (Pin_9)
- net GPI7: now reaches U1.9 (GPIO7)
- net GPI7: now also J2.10 (Pin_10)
- new net: R7.1, SW1.2
- new net: C16.2, R5.2, Y1.1
- no-connect marks 0 -> 1
Other:
- moved on the sheet: C13, C14, J1, R1, R2, U1, U2

Commit message: beep
Parts:
- C1, C10, C11, C12, C17, C2, C3, C4, C5, C6, C7, C8, C9: footprint (none) -> Capacitor_SMD:C_0402_1005Metric
- C13, C14: footprint (none) -> Capacitor_SMD:C_0603_1608Metric
- C15, C16: value 15pF -> 33pF; footprint (none) -> Capacitor_SMD:C_0402_1005Metric
- J1: footprint (none) -> Connector_USB:USB_C_Receptacle_HRO_TYPE-C-31-M-12
- J2, J3: footprint (none) -> Connector_PinHeader_2.54mm:PinHeader_1x20_P2.54mm_Vertical
- J4: footprint (none) -> Connector_PinHeader_2.54mm:PinHeader_1x03_P2.54mm_Vertical
- R1, R2, R3, R4, R6, R7: footprint (none) -> Resistor_SMD:R_0402_1005Metric
- R5: value R -> 1K; footprint (none) -> Resistor_SMD:R_0402_1005Metric
- SW1: footprint (none) -> Button_Switch_SMD:SW_Push_SPST_NO_Alps_SKRK
- Y1: footprint (none) -> Crystal:Crystal_SMD_3225-4Pin_3.2x2.5mm
Changed lines of the file:
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@@
 			)
 		)
-		(property "Footprint" ""
+		(property "Footprint" "Capacitor_SMD:C_0402_1005Metric"
 			(at 204.1652 34.29 0)
 			(effects
@@
 			)
 		)
-		(property "Footprint" ""
+		(property "Footprint" "Capacitor_SMD:C_0402_1005Metric"
 			(at 134.3152 34.29 0)
 			(effects
@@
 			)
 		)
-		(property "Footprint" ""
+		(property "Footprint" "Capacitor_SMD:C_0402_1005Metric"
 			(at 172.4152 34.29 0)
 			(effects
@@
 			)
 		)
-		(property "Footprint" ""
+		(property "Footprint" "Connector_PinHeader_2.54mm:PinHeader_1x20_P2.54mm_Vertical"
 			(at 40.64 147.32 0)
 			(effects
@@
 			)
 		)
-		(property "Footprint" ""
+		(property "Footprint" "Resistor_SMD:R_0402_1005Metric"
 			(at 57.15 33.782 90)
 			(effects
@@
 			)
 		)
-		(property "Footprint" ""
+		(property "Footprint" "Resistor_SMD:R_0402_1005Metric"
 			(at 57.15 31.242 90)
 			(effects
@@
 			)
 		)
-		(property "Footprint" ""
+		(property "Footprint" "Connector_PinHeader_2.54mm:PinHeader_1x03_P2.54mm_Vertical"
 			(at 57.15 173.99 0)
 			(effects
@@
 			)
 		)
-		(property "Footprint" ""
+		(property "Footprint" "Capacitor_SMD:C_0402_1005Metric"
 			(at 159.7152 34.29 0)
 			(effects
@@
 			)
 		)
-		(property "Footprint" ""
+		(property "Footprint" "Resistor_SMD:R_0402_1005Metric"
 			(at 223.52 70.358 90)
 			(effects
@@
 			)
 		)
-		(property "Footprint" ""
+		(property "Footprint" "Button_Switch_SMD:SW_Push_SPST_NO_Alps_SKRK"
 			(at 210.82 63.5 0)
 			(effects
@@
 			)
 		)
-		(property "Footprint" ""
+		(property "Footprint" "Resistor_SMD:R_0402_1005Metric"
 			(at 123.19 84.582 90)
 			(effects
@@
 			)
 		)
-		(property "Footprint" ""
+		(property "Footprint" "Capacitor_SMD:C_0402_1005Metric"
 			(at 140.6652 34.29 0)
 			(effects
@@
 			)
 		)
-		(property "Footprint" ""
+		(property "Footprint" "Resistor_SMD:R_0402_1005Metric"
 			(at 123.19 87.122 90)
 			(effects
@@
 			)
 		)
-		(property "Footprint" ""
+		(property "Footprint" "Capacitor_SMD:C_0603_1608Metric"
 			(at 91.1352 35.56 0)
 			(effects
@@
 			)
 		)
-		(property "Footprint" ""
+		(property "Footprint" "Connector_USB:USB_C_Receptacle_HRO_TYPE-C-31-M-12"
 			(at 40.64 43.18 0)
 			(effects
@@
 			)
 		)
-		(property "Footprint" ""
+		(property "Footprint" "Capacitor_SMD:C_0402_1005Metric"
 			(at 147.0152 34.29 0)
 			(effects
@@
 			)
 		)
-		(property "Value" "15pF"
+		(property "Value" "33pF"
 			(at 224.79 123.698 0)
 			(effects
@@
 			)
 		)
-		(property "Footprint" ""
+		(property "Footprint" "Capacitor_SMD:C_0402_1005Metric"
 			(at 226.06 123.4948 0)
 			(effects
@@
 			)
 		)
-		(property "Value" "15pF"
+		(property "Value" "33pF"
 			(at 224.79 135.128 0)
 			(effects
@@
 			)
 		)
-		(property "Footprint" ""
+		(property "Footprint" "Capacitor_SMD:C_0402_1005Metric"
 			(at 226.06 134.9248 0)
 			(effects
@@
 			)
 		)
-		(property "Footprint" ""
+		(property "Footprint" "Crystal:Crystal_SMD_3225-4Pin_3.2x2.5mm"
 			(at 234.95 129.54 0)
 			(effects
@@
 			)
 		)
-		(property "Footprint" ""
+		(property "Footprint" "Capacitor_SMD:C_0402_1005Metric"
 			(at 197.8152 34.29 0)
 			(effects
@@
 			)
 		)
-		(property "Footprint" ""
+		(property "Footprint" "Capacitor_SMD:C_0603_1608Metric"
 			(at 69.5452 35.56 0)
 			(effects
@@
 			)
 		)
-		(property "Footprint" ""
+		(property "Footprint" "Capacitor_SMD:C_0402_1005Metric"
 			(at 185.1152 34.29 0)
 			(effects
@@
 			)
 		)
-		(property "Footprint" ""
+		(property "Footprint" "Resistor_SMD:R_0402_1005Metric"
 			(at 230.632 62.23 90)
 			(effects
@@
 			)
 		)
-		(property "Footprint" ""
+		(property "Footprint" "Capacitor_SMD:C_0402_1005Metric"
 			(at 178.7652 34.29 0)
 			(effects
@@
 			)
 		)
-		(property "Footprint" ""
+		(property "Footprint" "Capacitor_SMD:C_0402_1005Metric"
 			(at 210.5152 34.29 0)
 			(effects
@@
 			)
 		)
-		(property "Footprint" ""
+		(property "Footprint" "Capacitor_SMD:C_0402_1005Metric"
 			(at 166.0652 34.29 0)
 			(effects
@@
 			)
 		)
-		(property "Footprint" ""
+		(property "Footprint" "Capacitor_SMD:C_0402_1005Metric"
 			(at 264.16 57.4548 0)
 			(effects
@@
 			)
 		)
-		(property "Footprint" ""
+		(property "Footprint" "Capacitor_SMD:C_0402_1005Metric"
 			(at 191.4652 34.29 0)
 			(effects
@@
 			)
 		)
-		(property "Footprint" ""
+		(property "Footprint" "Connector_PinHeader_2.54mm:PinHeader_1x20_P2.54mm_Vertical"
 			(at 72.39 147.32 0)
 			(effects
@@
 		(on_board yes)
 		(dnp no)
-		(fields_autoplaced yes)
 		(property "Reference" "R5"
-			(at 248.92 129.54 90)
+			(at 248.92 130.556 90)
 			(effects
 				(font
@@
 			)
 		)
-		(property "Value" "R"
-			(at 248.92 132.08 90)
+		(property "Value" "1K"
+			(at 248.92 133.096 90)
 			(effects
 				(font
@@
 			)
 		)
-		(property "Footprint" ""
+		(property "Footprint" "Resistor_SMD:R_0402_1005Metric"
 			(at 248.92 134.112 90)
 			(effects

Commit message: b
Parts:
- U3: value W25Q128JVS -> W25Q16JVZPIQ TR; footprint Package_SO:SOIC-8_5.3x5.3mm_P1.27mm -> Package_SON:Winbond_USON-8-1EP_3x2mm_P0.5mm_EP0.2x1.6mm
Changed lines of the file:
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@@
 			)
 		)
-		(property "Value" "W25Q128JVS"
+		(property "Value" "W25Q16JVZPIQ TR"
 			(at 266.7 77.4699 0)
 			(effects
@@
 			)
 		)
-		(property "Footprint" "Package_SO:SOIC-8_5.3x5.3mm_P1.27mm"
+		(property "Footprint" "Package_SON:Winbond_USON-8-1EP_3x2mm_P0.5mm_EP0.2x1.6mm"
 			(at 255.27 53.34 0)
 			(effects
