File: catboard/catboard.kicad_pcb (KiCad board)
At the start: 2 copper layers, 21 x 51 mm, 33 parts, among them J1 USB_C_Receptacle_USB2.0_14P, J2 Conn_01x20, J3 Conn_01x20, J4 Conn_01x03, SW1 SW_Push, U1 RP2040, U2 MCP1700x-330xxTT, U3 W25Q16JVZPIQ TR, Y1 12 MHz

Commit message: badoop
Parts:
- moved R7 21.0 mm to (171.8, 91.0)
- moved R5 19.1 mm to (168.3, 112.8), turned to 0 degrees
- moved SW1 3.09 mm to (171.8, 87.7)
- moved C1 1.79 mm to (172.8, 99.8)
- moved C12 1.35 mm to (162.0, 108.5), turned to -135 degrees
- moved C6 1.23 mm to (169.0, 98.1)
- moved C9 1.23 mm to (168.0, 98.1)
- moved C7 1.23 mm to (170.0, 97.5)
- moved C10 1.12 mm to (170.9, 113.2)
- moved C16 1.12 mm to (169.9, 115.1)
- moved C2 1.12 mm to (169.9, 113.2)
- moved C15 1.12 mm to (164.5, 115.1)
- moved Y1 1.12 mm to (167.2, 115.1), turned to 180 degrees
- moved R3 1.10 mm to (169.7, 101.3), turned to 90 degrees
- moved C4 0.92 mm to (163.7, 102.2)
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Routing:
- net +3V3: track 0.00 -> 88.8 mm, vias 0 -> 7
- net GND: track 0.00 -> 45.6 mm, vias 0 -> 6
- net GPI0: track 0.00 -> 35.9 mm, vias 0 -> 1
- net GPI1: track 0.00 -> 27.0 mm, vias 0 -> 1
- net GPI29_ADC3: track 0.00 -> 26.5 mm, vias 0 -> 2
- net QSPI_SS: track 0.00 -> 24.0 mm, vias 0 -> 2
- net SWCLK: track 0.00 -> 23.3 mm
- net GPI2: track 0.00 -> 22.7 mm, vias 0 -> 1
- net USB_D+: track 0.00 -> 22.6 mm
- net USB_D-: track 0.00 -> 22.6 mm
- net GPI28_ADC2: track 0.00 -> 22.3 mm
- net GPI16: track 0.00 -> 21.9 mm
- net GPI3: track 0.00 -> 20.4 mm
- net GPI15: track 0.00 -> 20.2 mm
- net VBUS: track 0.00 -> 20.1 mm
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- added copper zone on B.Cu, net GND
- added copper zone on F.Cu, net GND
Other:
- board size 21 x 51 mm -> 21.5 x 51.8 mm

Commit message: bbb
Routing:
- net GND: track 45.6 -> 59.8 mm, vias 6 -> 11
