File: pcb/catboard.kicad_pcb (KiCad board)
At the start: 2 copper layers, 21.5 x 51.8 mm, 33 parts, among them J1 USB_C_Receptacle_USB2.0_14P, J2 Conn_01x20, J3 Conn_01x20, J4 Conn_01x03, SW1 SW_Push, U1 RP2040, U2 MCP1700x-330xxTT, U3 W25Q16JVZPIQ TR, Y1 12 MHz

Commit message: boooop
Parts:
- U3: value W25Q16JVZPIQ TR -> W25Q128JVP; footprint Package_SON:Winbond_USON-8-1EP_3x2mm_P0.5mm_EP0.2x1.6mm -> Package_SON:WSON-8-1EP_6x5mm_P1.27mm_EP3.4x4.3mm
- moved C17 4.50 mm to (166.5, 92.7)
- moved R6 4.50 mm to (164.5, 92.7)
- moved C7 3.33 mm to (172.0, 94.9)
- moved U3 3.26 mm to (165.8, 96.0)
- moved C6 3.25 mm to (171.0, 95.5)
- moved C9 3.25 mm to (170.0, 95.5)
Connections:
- U3 pad 9: (no net) -> GND
Routing:
- net GND: track 59.8 -> 90.5 mm, vias 11 -> 18
- net +3V3: track 88.8 -> 80.3 mm
- net QSPI_SD3: track 5.45 -> 9.31 mm
- net USB_D+: track 22.6 -> 26.4 mm
- net USB_D-: track 22.6 -> 26.3 mm
- net QSPI_SCLK: track 4.50 -> 7.88 mm
- net QSPI_SD1: track 8.01 -> 10.9 mm
- net QSPI_SD0: track 3.56 -> 5.97 mm
- net QSPI_SD2: track 6.60 -> 8.47 mm
- net QSPI_SS: track 24.1 -> 25.9 mm
- net GPI0: track 35.9 -> 36.7 mm
