File: pcb/catboard.kicad_sch (KiCad schematic)
At the start: 33 parts, among them J1 USB_C_Receptacle_USB2.0_14P, J2 Conn_01x20, J3 Conn_01x20, J4 Conn_01x03, SW1 SW_Push, U1 RP2040, U2 MCP1700x-330xxTT, U3 W25Q16JVZPIQ TR, Y1 12 MHz

Commit message: boooop
Parts:
- removed U3: W25Q16JVZPIQ TR, Package_SON:Winbond_USON-8-1EP_3x2mm_P0.5mm_EP0.2x1.6mm, symbol Memory_Flash:W25Q128JVS
- added U3: W25Q128JVP, Package_SON:WSON-8-1EP_6x5mm_P1.27mm_EP3.4x4.3mm, symbol Memory_Flash:W25Q128JVP
Connections:
- net +3V3: now also U3.8 (VCC)
- net GND: now also U3.4 (GND), U3.9 (EP)
- net QSPI_SCLK: now also U3.6 (CLK)
- net QSPI_SD0: now also U3.5 (DI/IO_{0})
- net QSPI_SD1: now also U3.2 (DO/IO_{1})
- net QSPI_SD2: now also U3.3 (~{WP}/IO_{2})
- net QSPI_SD3: now also U3.7 (~{HOLD}/~{RESET}/IO_{3})
- net QSPI_SS: now also U3.1 (~{CS})
Changed lines of the file:
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@@
 	(wire
 		(pts
+			(xy 257.81 88.9) (xy 260.35 88.9)
+		)
+		(stroke
+			(width 0)
+			(type default)
+		)
+	)
+	(wire
+		(pts
 			(xy 234.95 133.35) (xy 234.95 135.89)
 		)
@@
 	(wire
 		(pts
+			(xy 260.35 88.9) (xy 260.35 90.17)
+		)
+		(stroke
+			(width 0)
+			(type default)
+		)
+	)
+	(wire
+		(pts
 			(xy 125.73 137.16) (xy 128.27 137.16)
 		)
@@
 	)
 	(symbol
+		(lib_id "power:GND")
+		(at 260.35 90.17 0)
+		(unit 1)
+		(exclude_from_sim no)
+		(in_bom yes)
+		(on_board yes)
+		(dnp no)
+		(fields_autoplaced yes)
+		(property "Reference" "#PWR027"
+			(at 260.35 96.52 0)
+			(effects
+				(font
+					(size 1.27 1.27)
+				)
+				(hide yes)
+			)
+		)
+		(property "Value" "GND"
+			(at 260.35 95.25 0)
+			(effects
+				(font
+					(size 1.27 1.27)
+				)
+			)
+		)
+		(property "Footprint" ""
+			(at 260.35 90.17 0)
+			(effects
+				(font
+					(size 1.27 1.27)
+				)
+				(hide yes)
+			)
+		)
+		(property "Datasheet" ""
+			(at 260.35 90.17 0)
+			(effects
+				(font
+					(size 1.27 1.27)
+				)
+				(hide yes)
+			)
+		)
+		(property "Description" "Power symbol creates a global label with name \"GND\" , ground"
+			(at 260.35 90.17 0)
+			(effects
+				(font
+					(size 1.27 1.27)
+				)
+				(hide yes)
+			)
+		)
+		(pin "1"
+		)
+		(instances
+			(project ""
+				(path "/902a8887-3e18-4426-bd46-bd30446d4a6d"
+					(reference "#PWR027")
+					(unit 1)
+				)
+			)
+		)
+	)
+	(symbol
 		(lib_id "power:+3V3")
 		(at 97.79 26.67 0)
@@
 	)
 	(symbol
-		(lib_id "Regulator_Linear:MCP1700x-330xxTT")
-		(at 80.01 27.94 0)
+		(lib_id "Memory_Flash:W25Q128JVP")
+		(at 255.27 76.2 0)
 		(unit 1)
 		(exclude_from_sim no)
@@
 		(dnp no)
 		(fields_autoplaced yes)
-		(property "Reference" "U2"
-			(at 80.01 21.59 0)
+		(property "Reference" "U3"
+			(at 266.7 74.9299 0)
 			(effects
 				(font
 					(size 1.27 1.27)
 				)
+				(justify left)
 			)
 		)
-		(property "Value" "MCP1700x-330xxTT"
-			(at 80.01 24.13 0)
+		(property "Value" "W25Q128JVP"
+			(at 266.7 77.4699 0)
 			(effects
 				(font
 					(size 1.27 1.27)
 				)
+				(justify left)
 			)
 		)
-		(property "Footprint" "Package_TO_SOT_SMD:SOT-23"
-			(at 80.01 22.225 0)
+		(property "Footprint" "Package_SON:WSON-8-1EP_6x5mm_P1.27mm_EP3.4x4.3mm"
+			(at 255.27 53.34 0)
 			(effects
 				(font
@@
 			)
 		)
-		(property "Datasheet" "http://ww1.microchip.com/downloads/en/DeviceDoc/20001826D.pdf"
-			(at 80.01 27.94 0)
+		(property "Datasheet" "https://www.winbond.com/resource-files/w25q128jv_dtr%20revc%2003272018%20plus.pdf"
+			(at 255.27 50.8 0)
 			(effects
 				(font
@@
 			)
 		)
-		(property "Description" "250mA Low Quiscent Current LDO, 3.3V output, SOT-23"
-			(at 80.01 27.94 0)
+		(property "Description" "128Mbit / 16MiB Serial Flash Memory, Standard/Dual/Quad SPI, 2.7-3.6V, WSON-8"
+			(at 255.27 48.26 0)
 			(effects
 				(font
@@
 			)
 		)
-		(pin "1"
+		(pin "5"
 		)
 		(pin "2"
@@
 		(pin "3"
 		)
+		(pin "7"
+		)
+		(pin "8"
+		)
+		(pin "4"
+		)
+		(pin "9"
+		)
+		(pin "6"
+		)
+		(pin "1"
+		)
 		(instances
 			(project ""
 				(path "/902a8887-3e18-4426-bd46-bd30446d4a6d"
-					(reference "U2")
+					(reference "U3")
 					(unit 1)
 				)
@@
 	)
 	(symbol
-		(lib_id "Memory_Flash:W25Q128JVS")
-		(at 255.27 76.2 0)
+		(lib_id "Regulator_Linear:MCP1700x-330xxTT")
+		(at 80.01 27.94 0)
 		(unit 1)
 		(exclude_from_sim no)
@@
 		(dnp no)
 		(fields_autoplaced yes)
-		(property "Reference" "U3"
-			(at 266.7 74.9299 0)
+		(property "Reference" "U2"
+			(at 80.01 21.59 0)
 			(effects
 				(font
 					(size 1.27 1.27)
 				)
-				(justify left)
 			)
 		)
-		(property "Value" "W25Q16JVZPIQ TR"
-			(at 266.7 77.4699 0)
+		(property "Value" "MCP1700x-330xxTT"
+			(at 80.01 24.13 0)
 			(effects
 				(font
 					(size 1.27 1.27)
 				)
-				(justify left)
 			)
 		)
-		(property "Footprint" "Package_SON:Winbond_USON-8-1EP_3x2mm_P0.5mm_EP0.2x1.6mm"
-			(at 255.27 53.34 0)
+		(property "Footprint" "Package_TO_SOT_SMD:SOT-23"
+			(at 80.01 22.225 0)
 			(effects
 				(font
@@
 			)
 		)
-		(property "Datasheet" "https://www.winbond.com/resource-files/w25q128jv_dtr%20revc%2003272018%20plus.pdf"
-			(at 255.27 50.8 0)
+		(property "Datasheet" "http://ww1.microchip.com/downloads/en/DeviceDoc/20001826D.pdf"
+			(at 80.01 27.94 0)
 			(effects
 				(font
@@
 			)
 		)
-		(property "Description" "128Mbit / 16MiB Serial Flash Memory, Standard/Dual/Quad SPI, 2.7-3.6V, SOIC-8"
-			(at 255.27 48.26 0)
+		(property "Description" "250mA Low Quiscent Current LDO, 3.3V output, SOT-23"
+			(at 80.01 27.94 0)
 			(effects
 				(font
@@
 			)
 		)
-		(pin "4"
+		(pin "1"
 		)
 		(pin "2"
 		)
-		(pin "8"
-		)
 		(pin "3"
 		)
-		(pin "7"
-		)
-		(pin "6"
-		)
-		(pin "5"
-		)
-		(pin "1"
-		)
 		(instances
 			(project ""
 				(path "/902a8887-3e18-4426-bd46-bd30446d4a6d"
-					(reference "U3")
+					(reference "U2")
 					(unit 1)
 				)
